File: FringeLocker/FringeLocker.sch (KiCad schematic (older format))
At the start: 16 parts, among them J1 Conn_Piezo, U1 TL072

Commit message: started PCB
Parts:
- C1, C2: footprint (none) -> Capacitor_THT:CP_Radial_D5.0mm_P2.00mm
- C3: footprint (none) -> Capacitor_THT:CP_Radial_Tantal_D4.5mm_P5.00mm
Changed lines of the file:
@@
 F 0 "C1" V 6952 3800 50  0000 C CNN
 F 1 "1uF" V 6861 3800 50  0000 C CNN
-F 2 "" H 6738 3650 50  0001 C CNN
+F 2 "Capacitor_THT:CP_Radial_D5.0mm_P2.00mm" H 6738 3650 50  0001 C CNN
 F 3 "~" H 6700 3800 50  0001 C CNN
 	1    6700 3800
@@
 F 0 "C2" V 6952 4400 50  0000 C CNN
 F 1 "1uF" V 6861 4400 50  0000 C CNN
-F 2 "" H 6738 4250 50  0001 C CNN
+F 2 "Capacitor_THT:CP_Radial_D5.0mm_P2.00mm" H 6738 4250 50  0001 C CNN
 F 3 "~" H 6700 4400 50  0001 C CNN
 	1    6700 4400
@@
 F 0 "C3" V 7400 2150 50  0000 C CNN
 F 1 "1.6nF" V 7300 2100 50  0000 C CNN
-F 2 "" H 7388 2100 50  0001 C CNN
+F 2 "Capacitor_THT:CP_Radial_Tantal_D4.5mm_P5.00mm" H 7388 2100 50  0001 C CNN
 F 3 "~" H 7350 2250 50  0001 C CNN
 	1    7350 2250
