File: FringeLocker/FringeLocker.kicad_pcb (KiCad board)
At the start: 2 copper layers, 17 parts, among them J1 OUT, J2 PWR, U1 TL072

Commit message: V1.0
Parts:
- added BH1: KeysTone_AAA, BatteryHolder:Keystone_AAA, F.Cu at (158.8, 75.5)
- added BH2: KeysTone_AAA, BatteryHolder:Keystone_AAA, F.Cu at (116.7, 84.5)
- added C4: 160nF, Capacitor_SMD:C_0603_1608Metric_Pad1.08x0.95mm_HandSolder, B.Cu at (132.9, 82.2)
- added C5: 1uF, Capacitor_SMD:C_0603_1608Metric_Pad1.08x0.95mm_HandSolder, B.Cu at (142.0, 76.3)
- added C6: 1uF, Capacitor_SMD:C_0603_1608Metric_Pad1.08x0.95mm_HandSolder, B.Cu at (148.5, 76.0)
- added D3: LED_Small, LED_SMD:LED_0402_1005Metric_Pad0.77x0.64mm_HandSolder, F.Cu at (141.6, 102.8)
- added J3: Conn_01x03_Male, Connector_PinHeader_2.54mm:PinHeader_1x03_P2.54mm_Vertical, F.Cu at (147.4, 100.9)
- added R10: 10K, Resistor_SMD:R_0805_2012Metric_Pad1.20x1.40mm_HandSolder, B.Cu at (143.0, 102.8)
- added R8: 10K, Resistor_SMD:R_0805_2012Metric_Pad1.20x1.40mm_HandSolder, B.Cu at (130.8, 78.0)
- added R9: 1K, Resistor_SMD:R_0805_2012Metric_Pad1.20x1.40mm_HandSolder, B.Cu at (130.8, 82.1)
- added REF1: MountingHole_2.2mm_M2_DIN965_Pad, MountingHole:MountingHole_2.2mm_M2_DIN965_Pad, F.Cu at (109.5, 56.5)
- added REF2: MountingHole_2.2mm_M2_DIN965_Pad, MountingHole:MountingHole_2.2mm_M2_DIN965_Pad, F.Cu at (164.5, 56.5)
- added REF3: MountingHole_2.2mm_M2_DIN965_Pad, MountingHole:MountingHole_2.2mm_M2_DIN965_Pad, F.Cu at (164.5, 104.5)
- added REF4: MountingHole_2.2mm_M2_DIN965_Pad, MountingHole:MountingHole_2.2mm_M2_DIN965_Pad, F.Cu at (109.5, 104.5)
- added SW1: NIDEC_SS-10-16, BatteryHolder:NIDEC_SS-10-16, F.Cu at (128.1, 73.1)
- added SW2: SW_Push_DPDT, BatteryHolder:SlideSwitchASE_DPDT, F.Cu at (131.7, 104.4)
- added TP1: TP OUT, TestPoint:TestPoint_THTPad_D1.0mm_Drill0.5mm, F.Cu at (134.3, 94.2)
- added TP2: TP Bias, TestPoint:TestPoint_THTPad_D1.0mm_Drill0.5mm, F.Cu at (158.4, 101.5)
- added TP3: TP PDs, TestPoint:TestPoint_THTPad_D1.0mm_Drill0.5mm, F.Cu at (137.6, 65.2)
- C1: value 1uF -> 160pF; footprint Capacitor_THT:CP_Radial_D5.0mm_P2.00mm -> Capacitor_SMD:C_0603_1608Metric_Pad1.08x0.95mm_HandSolder; moved to B.Cu
- C2: value 1uF -> 1.6nF; footprint Capacitor_THT:CP_Radial_D5.0mm_P2.00mm -> Capacitor_SMD:C_0603_1608Metric_Pad1.08x0.95mm_HandSolder; moved to B.Cu
- C3: value 1.6nF -> 16nF; footprint Capacitor_THT:CP_Radial_Tantal_D4.5mm_P5.00mm -> Capacitor_SMD:C_0603_1608Metric_Pad1.08x0.95mm_HandSolder; moved to B.Cu
- D1, D2: moved to B.Cu
- J2: value PWR -> TP Scaler; footprint Connector_PinHeader_2.54mm:PinHeader_1x03_P2.54mm_Vertical -> Connector_PinHeader_2.54mm:PinHeader_1x02_P2.54mm_Vertical
- R1, R2: footprint Resistor_THT:R_Axial_DIN0207_L6.3mm_D2.5mm_P10.16mm_Horizontal -> Resistor_SMD:R_0805_2012Metric_Pad1.20x1.40mm_HandSolder; moved to B.Cu
- R3: value 1K -> 100K; footprint Resistor_THT:R_Axial_DIN0207_L6.3mm_D2.5mm_P10.16mm_Horizontal -> Resistor_SMD:R_0805_2012Metric_Pad1.20x1.40mm_HandSolder; moved to B.Cu
- R4: value 100K -> 1K; footprint Resistor_THT:R_Axial_DIN0207_L6.3mm_D2.5mm_P10.16mm_Horizontal -> Resistor_SMD:R_0805_2012Metric_Pad1.20x1.40mm_HandSolder; moved to B.Cu
- R5: value 10K -> 100K; footprint Resistor_THT:R_Axial_DIN0207_L6.3mm_D2.5mm_P10.16mm_Horizontal -> Resistor_SMD:R_0805_2012Metric_Pad1.20x1.40mm_HandSolder; moved to B.Cu
- R6: value 10K -> 1M; footprint Resistor_THT:R_Axial_DIN0207_L6.3mm_D2.5mm_P10.16mm_Horizontal -> Resistor_SMD:R_0805_2012Metric_Pad1.20x1.40mm_HandSolder; moved to B.Cu
- R7: value 4.7K -> 100K; footprint Resistor_THT:R_Axial_DIN0207_L6.3mm_D2.5mm_P10.16mm_Horizontal -> Resistor_SMD:R_0805_2012Metric_Pad1.20x1.40mm_HandSolder; moved to B.Cu
- RV1: footprint Potentiometer_THT:Potentiometer_Bourns_3386F_Vertical -> Potentiometer_THT:Potentiometer_Bourns_3266W_Vertical
- RV2: value 10K -> 100K; footprint Potentiometer_THT:Potentiometer_Bourns_3386F_Vertical -> Potentiometer_THT:Potentiometer_Bourns_3266W_Vertical
- U1: value TL072 -> TL074; footprint Package_SO:SOIC-8_3.9x4.9mm_P1.27mm -> Package_SO:SO-14_5.3x10.2mm_P1.27mm
- moved D2 65.3 mm to (138.5, 59.0), turned to 0 degrees
- moved D1 64.3 mm to (131.0, 59.0), turned to 0 degrees
- moved C2 48.0 mm to (132.9, 74.0), turned to -90 degrees
- moved C1 44.3 mm to (132.9, 69.7), turned to -90 degrees
- moved R6 42.4 mm to (130.8, 69.8)
- moved R1 37.7 mm to (141.1, 86.0), turned to -90 degrees
- moved J1 37.3 mm to (147.9, 90.2), turned to 0 degrees
- moved R3 37.3 mm to (145.2, 80.2), turned to -90 degrees
- moved U1 33.0 mm to (145.1, 76.3)
- moved R2 32.8 mm to (137.0, 86.1), turned to -90 degrees
- moved RV1 32.2 mm to (125.9, 89.8), turned to 180 degrees
- moved J2 31.0 mm to (120.5, 102.6), turned to 0 degrees
- moved R4 28.5 mm to (133.9, 88.5), turned to 90 degrees
- moved C3 26.1 mm to (132.9, 78.0)
- moved R5 22.7 mm to (145.3, 85.5), turned to 90 degrees
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Connections:
- C1 pad 1: +15V -> Net-(C1-Pad1)
- C1 pad 2: GND -> Net-(C1-Pad2)
- C2 pad 1: -15V -> Net-(C1-Pad1)
- C2 pad 2: GND -> Net-(C2-Pad2)
- C3 pad 1: Net-(C3-Pad1) -> Net-(C1-Pad1)
- D1 pad 2: Net-(R5-Pad1) -> Net-(D1-Pad2)
- D2 pad 1: Net-(R5-Pad1) -> Net-(D1-Pad2)
- J1 pad 2: -15V -> Net-(J1-Pad2)
- J2 pad 1: +15V -> Net-(C1-Pad1)
- R3 pad 2: Net-(R2-Pad1) -> Net-(J1-Pad2)
- R4 pad 1: Net-(C3-Pad2) -> Net-(R4-Pad1)
- R4 pad 2: Net-(C3-Pad1) -> Net-(R2-Pad1)
- R5 pad 2: Net-(C3-Pad2) -> Net-(R3-Pad1)
- R6 pad 1: Net-(C3-Pad2) -> Net-(C1-Pad2)
- R6 pad 2: Net-(R6-Pad2) -> Net-(C1-Pad1)
- R7 pad 1: Net-(R7-Pad1) -> Net-(C2-Pad2)
- R7 pad 2: +15V -> Net-(C1-Pad1)
- RV1 pad 1: Net-(C3-Pad1) -> Net-(C1-Pad1)
- RV1 pad 2: Net-(C3-Pad1) -> Net-(C1-Pad1)
- RV1 pad 3: Net-(R3-Pad1) -> Net-(R4-Pad1)
- RV2 pad 1: GND -> -15V
- RV2 pad 2: Net-(R6-Pad2) -> Net-(R5-Pad1)
- RV2 pad 3: Net-(R7-Pad1) -> +15V
- U1 pad 1: Net-(C3-Pad1) -> Net-(C1-Pad1)
- U1 pad 2: Net-(C3-Pad2) -> Net-(D1-Pad2)
- U1 pad 4: -15V -> +15V
- U1 pad 8: +15V -> Net-(J1-Pad2)
Routing:
- net GND: track 78.7 -> 0.00 mm
- net Net-(BH1-Pad1): track 0.00 -> 69.1 mm
- net Net-(BH2-Pad3): track 0.00 -> 63.2 mm
- net Net-(C1-Pad1): track 0.00 -> 61.7 mm, vias 0 -> 1
- net Net-(C3-Pad1): track 56.8 -> 0.00 mm
- net Net-(J1-Pad2): track 0.00 -> 41.8 mm
- net Net-(D1-Pad2): track 0.00 -> 32.7 mm
- net Net-(C3-Pad2): track 30.7 -> 6.15 mm
- net Net-(J1-Pad1): track 5.08 -> 24.9 mm
- net Net-(R3-Pad1): track 29.0 -> 9.35 mm, vias 0 -> 1
- net Net-(C4-Pad2): track 0.00 -> 16.9 mm
- net Net-(R5-Pad1): track 21.8 -> 6.11 mm
- net Net-(R7-Pad1): track 10.9 -> 0.00 mm
- net +15V: track 80.0 -> 90.5 mm, vias 0 -> 1
- net Net-(R6-Pad2): track 9.84 -> 0.00 mm
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- added copper zone on B.Cu, net GND
- added copper zone on F.Cu, net GND
Other:
- board outline added: 62.2 x 54.9 mm
- board text added: "+"
- board text added: "-"
- board text added: "Bias"
- board text added: "GND"
- board text added: "Gain"
- board text added: "Out"
- board text added: "PDs"
- board text added: "TP Scaler"
- board text added: "V+"
- board text added: "V-"
- board text added: "|<"
